File: pcb/microcontroller.kicad_sch (KiCad schematic)
At the start: 23 parts, among them J6 Conn_ARM_SWD_TagConnect_TC203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, SW1 SW_SPST, SW2 SW_SPST, SW3 SW_SPST, U3 W25Q16JVUXIQ TR, U4 RP2040, Y1 12MHz

Commit message: Prepped for DR
Parts:
- C10, C12, C13, C14, C4, C6, C7, C8: DPN 1276-1935-1-ND -> 1276-1938-1-ND; MPN CL10B104KB8NNWC -> CL10B104KO8NFNC
- C15: DPN 1276-1085-1-ND -> 1276-1938-1-ND; MPN CL10A225KP8NNNC -> CL10B104KO8NFNC
- C3: value 10u -> 22u; DPN GMC10X5R106M10NT -> 490-7611-1-ND; MPN 4713-GMC10X5R106M10NTCT-ND -> GRM188R60J226MEA0D
Connections:
- no-connect marks 6 -> 8

Commit message: Prepared for fab
Parts:
- renumbered C4 to C1, C15 to C10, C3 to C11, C5 to C12, C9 to C13, C7 to C2, C10 to C3, C12 to C4, C13 to C5, C14 to C6, C6 to C7, C11 to C9, D2 to D5, J6 to J9, R8 to R1, R6 to R2, SW2 to SW1, SW1 to SW2, U4 to U1, U3 to U2
Connections:
- net at U1.27 (GPIO16): no longer R1.2
- net at U1.37 (GPIO25): now also R1.2
Other:
- note added: "Boot"
- note added: "Reset"
- company: (none) -> Benjamin Crall
- title: (none) -> Breadboard Buddy
- moved on the sheet: D5, R1, SW2, SW3
